Commit message: use tf prefixes as 'prefix_link' instead of 'prefix/link'

File: mir_description/urdf/mir.urdf.xacro (robot description, xacro)
@@ -11,5 +11,5 @@
   </xacro:if>
   <xacro:unless value="${tf_prefix_ == ''}">
-    <xacro:property name="prefix" value="${tf_prefix_}/" />
+    <xacro:property name="prefix" value="${tf_prefix_}" />
   </xacro:unless>
   <xacro:mir prefix="${prefix}" />
